Commit message: cuTAMP changes for TiPToP

File: cutamp/robots/assets/ur5e_robotiq_2f_85.urdf (robot description, URDF)
Before this commit: robot robotiq_gripper, 24 links, 23 joints
Links:
- added link camera_mount, mass 0.05; collision mesh filename=assets/camera_mounts/ur5e_camera_mount.stl scale=0.001 0.001 0.001; visual mesh filename=assets/camera_mounts/ur5e_camera_mount.stl scale=0.001 0.001 0.001
Joints:
- added joint camera_mount_joint: type fixed, parent tool0, child camera_mount, origin xyz=0 0 0.0 rpy=0 0 0
- joint robotiq_85_base_joint: origin xyz=0 0 0 rpy=0 0 0 -> xyz=0 0 0.0 rpy=0 0 0; parent tool0 -> camera_mount
